Commit message: updated camera location

File: urdf/cobot_mimic.xacro (robot description, xacro)
@@ -67,5 +67,5 @@
      <!-- Define RGB-D sensor -->
     <xacro:kinetic_rgb name="rgbd_camera" parent="base">
-        <origin xyz="0.1 0.0 2.3" rpy="${0.0 * deg_to_rad} ${70.0 * deg_to_rad} ${0.0 * deg_to_rad}"/>
+        <origin xyz="0.5 0.0 1.8" rpy="${0.0 * deg_to_rad} ${70.0 * deg_to_rad} ${0.0 * deg_to_rad}"/>
         <origin xyz="0 0 0" rpy="${-90 * deg_to_rad} ${0 * deg_to_rad} ${-90 * deg_to_rad}" />
     </xacro:kinetic_rgb>

Commit message: changed color of robot and object

File: urdf/cobot_mimic.xacro (robot description, xacro)
@@ -76,3 +76,31 @@
         </plugin>
     </gazebo>
+    <!-- Make the robot more fancy :)-->
+    <gazebo reference="base_link" >
+        <material>Gazebo/Blue</material>
+    </gazebo>
+    <gazebo reference="link1" >
+        <material>Gazebo/Yellow</material>
+    </gazebo>
+    <gazebo reference="link2" >
+        <material>Gazebo/Black</material>
+    </gazebo>
+    <gazebo reference="link3" >
+        <material>Gazebo/Yellow</material>
+    </gazebo>
+    <gazebo reference="link4" >
+        <material>Gazebo/Black</material>
+    </gazebo>
+    <gazebo reference="link5" >
+        <material>Gazebo/Yellow</material>
+    </gazebo>
+    <gazebo reference="gripper_connector" >
+        <material>Gazebo/Black</material>
+    </gazebo>
+    <gazebo reference="gripper_right" >
+        <material>Gazebo/Blue</material>
+    </gazebo>
+    <gazebo reference="gripper_left" >
+        <material>Gazebo/Blue</material>
+    </gazebo>
 </robot>

Commit message: camara position

File: urdf/cobot_mimic.xacro (robot description, xacro)
@@ -67,5 +67,6 @@
      <!-- Define RGB-D sensor -->
     <xacro:kinetic_rgb name="rgbd_camera" parent="base">
-        <origin xyz="0.5 0.0 1.8" rpy="${0.0 * deg_to_rad} ${70.0 * deg_to_rad} ${0.0 * deg_to_rad}"/>
+        <!--<origin xyz="0.5 0.0 1.8" rpy="${0.0 * deg_to_rad} ${70.0 * deg_to_rad} ${0.0 * deg_to_rad}"/>-->
+        <origin xyz="0.7 0.0 1.5" rpy="${0.0 * deg_to_rad} ${70.0 * deg_to_rad} ${0.0 * deg_to_rad}"/>
         <origin xyz="0 0 0" rpy="${-90 * deg_to_rad} ${0 * deg_to_rad} ${-90 * deg_to_rad}" />
     </xacro:kinetic_rgb>

Commit message: change camera position

File: urdf/cobot_mimic.xacro (robot description, xacro)
@@ -68,5 +68,6 @@
     <xacro:kinetic_rgb name="rgbd_camera" parent="base">
         <!--<origin xyz="0.5 0.0 1.8" rpy="${0.0 * deg_to_rad} ${70.0 * deg_to_rad} ${0.0 * deg_to_rad}"/>-->
-        <origin xyz="0.7 0.0 1.5" rpy="${0.0 * deg_to_rad} ${70.0 * deg_to_rad} ${0.0 * deg_to_rad}"/>
+        <!--<origin xyz="0.7 0.0 1.5" rpy="${0.0 * deg_to_rad} ${70.0 * deg_to_rad} ${0.0 * deg_to_rad}"/>-->
+        <origin xyz="1 0.0 1" rpy="${0.0 * deg_to_rad} ${90.0 * deg_to_rad} ${0.0 * deg_to_rad}"/>
         <origin xyz="0 0 0" rpy="${-90 * deg_to_rad} ${0 * deg_to_rad} ${-90 * deg_to_rad}" />
     </xacro:kinetic_rgb>
